File: Keyboard Default.sch (KiCad schematic (older format))
At the start: 11 parts, among them P1 CONN_01X05, P2 USB_B, P3 CONN_01X05, SW1 SW_PUSH, U1 MCU-AT90USB1286-MU(TQFP64)

Commit message: added capacitors
Parts:
- added C0, C1: 10pF, symbol CP1
- added C3, C4, C5, C6: 0.1uF, symbol CP1
- added C7, C8: 1uF, symbol CP1
- added Y0: Crystal_Small, symbol Crystal_Small
Connections:
- net at U1.23 (XTAL2): now also C0.1, Y0.1
- net at U1.24 (XTAL1): now also C1.1, Y0.2
- net at U1.62 (AREF): now also C3.2
- net at U1.7 (UCAP): now also C7.1
- new net GND: C0.2, C1.2, C3.1, C4.2, C5.2, C6.2, C7.2, C8.2
- new net VCC: C4.1, C5.1, C6.1
